Commit message: Change URDF joint directions

File: puppersim/data/pupper_v2a.urdf (robot description, URDF)
Before this commit: robot pupper_v2_dji, 17 links, 16 joints
Joints:
- joint leftFrontLegMotor: axis 0 1.0 0 -> 0 -1.0 0
- joint leftFrontLowerLegMotor: axis 1.0 0 0 -> -1.0 0 0
- joint leftFrontUpperLegMotor: axis -1.0 0 0 -> 1.0 0 0; limit lower=-4.45059 upper=1.309 effort=0 velocity=0 -> lower=-1.309 upper=4.45059 effort=0 velocity=0
- joint leftRearLegMotor: axis 0 1.0 0 -> 0 -1.0 0
- joint leftRearLowerLegMotor: axis 1.0 0 0 -> -1.0 0 0
- joint leftRearUpperLegMotor: axis -1.0 0 0 -> 1.0 0 0; limit lower=-4.45059 upper=1.309 effort=0 velocity=0 -> lower=-1.309 upper=4.45059 effort=0 velocity=0
- joint rightFrontLegMotor: axis 0 -1.0 0 -> 0 1.0 0
- joint rightFrontLowerLegMotor: axis 1.0 0 0 -> -1.0 0 0
- joint rightFrontUpperLegMotor: axis 1.0 0 0 -> -1.0 0 0; limit lower=-4.45059 upper=1.309 effort=0 velocity=0 -> lower=-1.309 upper=4.45059 effort=0 velocity=0
- joint rightRearLegMotor: axis 0 -1.0 0 -> 0 1.0 0
- joint rightRearLowerLegMotor: axis 1.0 0 0 -> -1.0 0 0
- joint rightRearUpperLegMotor: axis 1.0 0 0 -> -1.0 0 0; limit lower=-4.45059 upper=1.309 effort=0 velocity=0 -> lower=-1.309 upper=4.45059 effort=0 velocity=0

File: puppersim/data/pupper_v2b.urdf (robot description, URDF)
Before this commit: robot pupper_v2_dji, 17 links, 16 joints
Joints:
- joint leftFrontLegMotor: axis 0 1.0 0 -> 0 -1.0 0
- joint leftFrontLowerLegMotor: axis 1.0 0 0 -> -1.0 0 0
- joint leftFrontUpperLegMotor: axis -1.0 0 0 -> 1.0 0 0; limit lower=-4.45059 upper=1.309 effort=0 velocity=0 -> lower=-1.309 upper=4.45059 effort=0 velocity=0
- joint leftRearLegMotor: axis 0 1.0 0 -> 0 -1.0 0
- joint leftRearLowerLegMotor: axis 1.0 0 0 -> -1.0 0 0
- joint leftRearUpperLegMotor: axis -1.0 0 0 -> 1.0 0 0; limit lower=-4.45059 upper=1.309 effort=0 velocity=0 -> lower=-1.309 upper=4.45059 effort=0 velocity=0
- joint rightFrontLegMotor: axis 0 -1.0 0 -> 0 1.0 0
- joint rightFrontLowerLegMotor: axis 1.0 0 0 -> -1.0 0 0
- joint rightFrontUpperLegMotor: axis 1.0 0 0 -> -1.0 0 0; limit lower=-4.45059 upper=1.309 effort=0 velocity=0 -> lower=-1.309 upper=4.45059 effort=0 velocity=0
- joint rightRearLegMotor: axis 0 -1.0 0 -> 0 1.0 0
- joint rightRearLowerLegMotor: axis 1.0 0 0 -> -1.0 0 0
- joint rightRearUpperLegMotor: axis 1.0 0 0 -> -1.0 0 0; limit lower=-4.45059 upper=1.309 effort=0 velocity=0 -> lower=-1.309 upper=4.45059 effort=0 velocity=0
